File: Bench_Power_Supply/Bench power supply.kicad_pcb (KiCad board)
At the start: 2 copper layers, 112.8 x 69 mm, 38 parts, among them P2 Conn_WallPlug, Q1 FQP33N10, U1 L7812, U2 LM358, U3 LM317T

Commit message: Add files via upload
Parts:
- removed ?: , Aesthetics:QTECHKNOW-LOGO-LARGE-SILK
- added R6: 1.5k, Resistor_THT:R_Axial_DIN0414_L11.9mm_D4.5mm_P15.24mm_Horizontal, F.Cu at (192.7, 96.9)
- added U4: ~, Bench_Power_Supply:Volt_Amper_Meter_5_Cable, F.Cu at (191.3, 119.6)
- D1, D2: footprint LED:LED_3MM -> LED_THT:LED_D5.0mm
- moved C6 38.4 mm to (160.9, 76.2), turned to 180 degrees
- moved RV1 24.7 mm to (160.7, 114.5)
- moved C4 22.4 mm to (189.6, 66.7)
- moved D3 17.9 mm to (186.1, 82.4), turned to -90 degrees
- moved R8 9.75 mm to (179.2, 96.0)
- moved R5 8.66 mm to (172.4, 95.7)
- moved R4 8.20 mm to (141.8, 83.4), turned to 180 degrees
- moved RV3 7.45 mm to (155.2, 105.9)
- moved U3 6.48 mm to (165.9, 68.8)
- moved Q1 6.38 mm to (156.2, 69.5)
- moved >NAME 6.03 mm to (162.3, 65.5)
- moved C2 5.04 mm to (133.4, 75.5)
- moved U2 4.35 mm to (148.3, 83.2)
- moved C5 3.62 mm to (173.3, 108.3)
- moved D4 3.30 mm to (120.7, 115.7)
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Connections:
- net Net-(D3-A) renamed /Load_Red
- C4 pad 2: Net-(Q1-D) -> /Load_Yellow
- C5 pad 2: Net-(Q1-D) -> /Load_Yellow
- C6 pad 2: Net-(Q1-D) -> /Load_Yellow
- Q1 pad 2: Net-(Q1-D) -> /Load_Yellow
- Q1 pad 3: Net-(Q1-D) -> Net-(Q1-S)
- R5 pad 2: Net-(Q1-D) -> Net-(Q1-S)
- R8 pad 2: Net-(Q1-D) -> Net-(Q1-S)
- RV4 pad 2: Net-(Q1-D) -> /Load_Yellow
- RV4 pad 3: Net-(Q1-D) -> /Load_Yellow
- TP2 pad 1: Net-(Q1-D) -> /Load_Yellow
Routing:
- net Net-(#FLG01-pwr): track 0.00 -> 203.1 mm, vias 0 -> 4
- net /Load_Red: track 0.00 -> 174.3 mm
- net Net-(D1-A): track 0.00 -> 156.9 mm, vias 0 -> 2
- net GND: track 0.00 -> 147.7 mm
- net /Load_Yellow: track 0.00 -> 131.3 mm, vias 0 -> 2
- net Net-(D9-A): track 0.00 -> 70.7 mm
- net Net-(Q1-G): track 0.00 -> 45.1 mm
- net Net-(D4-A): track 0.00 -> 39.9 mm
- net Net-(U2A--): track 0.00 -> 35.8 mm
- net Net-(Q1-S): track 0.00 -> 29.3 mm
- net Net-(R7-Pad1): track 0.00 -> 25.2 mm
- net Net-(R4-Pad1): track 0.00 -> 23.5 mm
- net Net-(D6-A): track 0.00 -> 19.7 mm
- net Net-(R2-Pad1): track 0.00 -> 18.9 mm
- net Net-(F1-Pad2): track 0.00 -> 14.0 mm
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
Commit message: Add files via upload
Parts:
- removed >NAME: >VALUE, Electromechanical:HEATSINK_PRT-9576
- added xx: yyy, Electromechanical:HEATSINK_PRT-9576, F.Cu at (162.2, 65.1)
Connections:
- R6 pad 2: GND -> /5v_volt
- U4 pad 1: GND -> /5v_volt
Routing:
- net GND: track 147.7 -> 0.00 mm
- net /5v_volt: track 0.00 -> 38.2 mm

Commit message: Add files via upload
Routing:
- net GND: track 0.00 -> 43.0 mm
- net /Load_Red: track 174.3 -> 173.5 mm
Other:
- board size 112.8 x 69 mm -> 112.8 x 74.8 mm
