File: Bench_Power_Supply/Bench power supply.kicad_sch (KiCad schematic)
At the start: 36 parts, among them P2 Conn_WallPlug, Q1 FQP33N10, U1 L7812, U2 LM358, U3 LM317T

Commit message: Add files via upload
Parts:
- added R6: 1.5k, Resistor_THT:R_Axial_DIN0414_L11.9mm_D4.5mm_P15.24mm_Horizontal, symbol Device:R
- added U4: ~, Bench_Power_Supply:Volt_Amper_Meter_5_Cable, symbol Bench_Power_Supply:Volt_AM_Meter
- D1, D2: footprint LED:LED_5MM-KIT -> LED_THT:LED_D5.0mm
Connections:
- net GND: now also R6.2, U4.1 (+DC_Red), U4.5 (-GNDLOAD_Black)
- net at C1.1, C2.1, C4.1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: now also R6.1
- net Load_Red: now reaches C5.1, D3.2 (A), D9.1 (K), RV3.1, RV3.2, TP1.1, U3.2 (OUT)
- net Load_Red: now also U4.3 (+LOAD_Red)
- net Load_Yellow: now reaches C4.2, C5.2, C6.2, Q1.2 (D), RV4.2, RV4.3, TP2.1
- net Load_Yellow: now also U4.4 (LOAD_Yellow)
- new net Gnd_volt: U4.2 (-GND_Black)
Other:
- moved on the sheet: D1, R1, U2C

Commit message: Add files via upload
Connections:
- net GND: no longer R6.2, U4.1 (+DC_Red)
- new net 5v_volt: R6.2, U4.1 (+DC_Red)
Changed lines of the file:
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@@
   (junction (at 79.2734 115.57) (diameter 0) (color 0 0 0 0)
   )
-  (junction (at 110.5916 74.549) (diameter 0) (color 0 0 0 0)
-  )
   (junction (at 205.9432 55.626) (diameter 0) (color 0 0 0 0)
   )
@@
   )
   (junction (at 104.3686 55.626) (diameter 0) (color 0 0 0 0)
-  )
-  (junction (at 110.5916 115.57) (diameter 0) (color 0 0 0 0)
   )
   (junction (at 165.4048 115.5192) (diameter 0) (color 0 0 0 0)
@@
     (stroke (width 0) (type default))
   )
-  (wire (pts (xy 110.5916 115.57) (xy 114.4016 115.57))
-    (stroke (width 0) (type default))
-  )
   (wire (pts (xy 124.7648 86.0552) (xy 124.7648 115.5192))
     (stroke (width 0) (type default))
@@
     (stroke (width 0) (type default))
   )
-  (wire (pts (xy 110.5916 74.549) (xy 110.5916 115.57))
-    (stroke (width 0) (type default))
-  )
   (wire (pts (xy 53.086 92.71) (xy 58.928 92.71))
     (stroke (width 0) (type default))
@@
     (stroke (width 0) (type default))
   )
-  (wire (pts (xy 104.3686 115.57) (xy 110.5916 115.57))
+  (wire (pts (xy 104.3686 115.57) (xy 114.4016 115.57))
     (stroke (width 0) (type default))
   )
@@
     (effects (font (size 1.27 1.27) (thickness 0.254) bold (color 194 0 0 1)) (justify left bottom))
   )
-  (label "5v_volt" (at 110.5916 106.2482 270) (fields_autoplaced)
+  (label "5v_volt" (at 110.5916 74.5236 270) (fields_autoplaced)
     (effects (font (size 1.27 1.27) (color 194 0 0 1)) (justify right bottom))
   )
@@
   (symbol (lib_id "Device:R") (at 110.5916 70.739 0) (unit 1)
     (in_bom yes) (on_board yes) (dnp no)
-    (property "Reference" "R6" (at 106.5276 69.469 0)
-      (effects (font (size 1.27 1.27)) (justify left))
-    )
-    (property "Value" "1.5k" (at 105.7402 71.9328 0)
-      (effects (font (size 1.27 1.27)) (justify left))
-    )
+    (property "Reference" "R6" (at 106.3752 68.9356 0)
+      (effects (font (size 1.27 1.27)) (justify left))
+    )
+    (property "Value" "1.5k" (at 105.537 71.628 0)
+      (effects (font (size 1.27 1.27)) (justify left))
+    )

Commit message: Add files via upload
Connections:
- no-connect marks 3 -> 4
Changed lines of the file:
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@@
   (no_connect (at 155.448 36.068))
   (no_connect (at 155.448 41.148))
+  (no_connect (at 82.9818 40.9194))
   (wire (pts (xy 205.867 32.766) (xy 205.867 55.6006))
     (stroke (width 0) (type default))
